File: eagle/MoteinoMegaGPSSheild.sch (EAGLE design)
At the start: 20 parts, among them J1 BilgeSwitch, J2 Button, J3 LED, J4 SCREW_TERM, J5 DS18B20, J6 DS18B20_12-24V_VCC, J7 OKI-78SR-5/1.5, J8 5V, Q1 NDP6020P P-CHANNEL, Q2 IRF9Z14PBF, Q3 2N7000

Commit message: Update
Parts:
- removed J6: DS18B20_12-24V_VCC, SparkFun-Connectors:CONN_023.5MM-NO_SILK
- added R5: 27M, SparkFun-Resistors:1MOHM-HORIZ_KIT-1/6W-5%
- added R6: 3.3M, SparkFun-Resistors:1MOHM-HORIZ_KIT-1/6W-5%
- J4: value SCREW_TERM -> DS18B20
- J5: value DS18B20 -> DS18B20_12-24V_VCC
Connections:
- removed net D1: J4.2, MOTEINO_MEGA.D1
- new net A5: MOTEINO_MEGA.A5, R5.2, R6.2
- net 12-24V-VCC: now also J5.2, R5.1; no longer J6.2
- net D27: now also J4.2; no longer J5.2
- net D28: now also J5.1; no longer J6.1
- net GND: now also R6.1; no longer J5.1
Other:
- moved on the sheet: J4, J5
Changed lines of the file:
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@@
 <schematic xreflabel="%F%N/%S.%C%R" xrefpart="/%S.%C%R">
 <attributes>
-<attribute name="CNAME" value="MoteinoMega Ultimate GPS Sheild"/>
-<attribute name="CREVISION" value="0.5"/>
+<attribute name="CNAME" value="MoteinoMega ABoatMon Sheild"/>
+<attribute name="CREVISION" value="0.6"/>
 <attribute name="DESIGNER" value="greg.cope@gmail.com"/>
 </attributes>
@@
 <part name="SUPPLY6" library="supply2" deviceset="GND" device=""/>
 <part name="J3" library="SparkFun-Connectors" deviceset="CONN_02" device="3.5MM-NO_SILK" value="LED"/>
-<part name="J4" library="SparkFun-Connectors" deviceset="CONN_02" device="3.5MM-NO_SILK" value="SCREW_TERM"/>
-<part name="SUPPLY7" library="supply2" deviceset="GND" device=""/>
-<part name="J5" library="SparkFun-Connectors" deviceset="CONN_02" device="3.5MM-NO_SILK" value="DS18B20"/>
-<part name="J6" library="SparkFun-Connectors" deviceset="CONN_02" device="3.5MM-NO_SILK" value="DS18B20_12-24V_VCC"/>
+<part name="J4" library="SparkFun-Connectors" deviceset="CONN_02" device="3.5MM-NO_SILK" value="DS18B20"/>
+<part name="J5" library="SparkFun-Connectors" deviceset="CONN_02" device="3.5MM-NO_SILK" value="DS18B20_12-24V_VCC"/>
 <part name="SUPPLY8" library="supply2" deviceset="GND" device=""/>
 <part name="Q2" library="transistor-power" deviceset="IRF9530" device="" value="IRF9Z14PBF"/>
@@
 <part name="SUPPLY10" library="supply2" deviceset="GND" device=""/>
 <part name="J8" library="SparkFun-Connectors" deviceset="CONN_01" device="" value="5V"/>
+<part name="R5" library="SparkFun-Resistors" deviceset="1MOHM" device="-HORIZ_KIT-1/6W-5%" value="27M"/>
+<part name="R6" library="SparkFun-Resistors" deviceset="1MOHM" device="-HORIZ_KIT-1/6W-5%" value="3.3M"/>
+<part name="SUPPLY11" library="supply2" deviceset="GND" device=""/>
 </parts>
 <sheets>
@@
 <instance part="SUPPLY6" gate="GND" x="30.48" y="137.16"/>
 <instance part="J3" gate="G$1" x="17.78" y="139.7"/>
-<instance part="J4" gate="G$1" x="68.58" y="165.1"/>
-<instance part="SUPPLY7" gate="GND" x="81.28" y="157.48"/>
-<instance part="J5" gate="G$1" x="25.4" y="12.7"/>
-<instance part="J6" gate="G$1" x="25.4" y="25.4"/>
+<instance part="J4" gate="G$1" x="25.4" y="12.7"/>
+<instance part="J5" gate="G$1" x="25.4" y="25.4"/>
 <instance part="SUPPLY8" gate="GND" x="43.18" y="10.16"/>
 <instance part="Q2" gate="G$1" x="254" y="76.2"/>
@@
 <instance part="SUPPLY10" gate="GND" x="264.16" y="40.64"/>
 <instance part="J8" gate="G$1" x="205.74" y="27.94"/>
+<instance part="R5" gate="G$1" x="208.28" y="101.6" rot="R270"/>
+<instance part="R6" gate="G$1" x="208.28" y="78.74" rot="R90"/>
+<instance part="SUPPLY11" gate="GND" x="208.28" y="68.58"/>
 </instances>
 <busses>
@@
 </segment>
 <segment>
-<pinref part="J5" gate="G$1" pin="1"/>
+<pinref part="J4" gate="G$1" pin="1"/>
 <pinref part="SUPPLY8" gate="GND" pin="GND"/>
 <wire x1="33.02" y1="12.7" x2="43.18" y2="12.7" width="0.1524" layer="91"/>
@@
 </segment>
 <segment>
-<pinref part="J4" gate="G$1" pin="1"/>
-<wire x1="76.2" y1="165.1" x2="81.28" y2="165.1" width="0.1524" layer="91"/>
-<pinref part="SUPPLY7" gate="GND" pin="GND"/>
-<wire x1="81.28" y1="165.1" x2="81.28" y2="160.02" width="0.1524" layer="91"/>
-</segment>
-<segment>
 <pinref part="Q3" gate="G$1" pin="S"/>
 <pinref part="SUPPLY9" gate="GND" pin="GND"/>
@@
 <pinref part="SUPPLY10" gate="GND" pin="GND"/>
 <wire x1="246.38" y1="43.18" x2="264.16" y2="43.18" width="0.1524" layer="91"/>
+</segment>
+<segment>
+<pinref part="R6" gate="G$1" pin="1"/>
+<wire x1="208.28" y1="73.66" x2="208.28" y2="71.12" width="0.1524" layer="91"/>
+<pinref part="SUPPLY11" gate="GND" pin="GND"/>
 </segment>
 </net>
@@
 </segment>
 </net>
-<net name="D1" class="0">
-<segment>
-<pinref part="J4" gate="G$1" pin="2"/>
-<wire x1="78.74" y1="167.64" x2="76.2" y2="167.64" width="0.1524" layer="91"/>
-<label x="15.24" y="160.02" size="1.778" layer="95"/>
-<label x="76.2" y="167.64" size="1.778" layer="95"/>
-</segment>
-<segment>
-<pinref part="MOTEINO_MEGA" gate="G$1" pin="D1"/>
-<wire x1="55.88" y1="106.68" x2="53.34" y2="106.68" width="0.1524" layer="91"/>
-<label x="53.34" y="106.68" size="1.778" layer="95"/>
-</segment>
-</net>
 <net name="12-24V-VCC" class="0">
 <segment>
-<pinref part="J6" gate="G$1" pin="2"/>
+<pinref part="J5" gate="G$1" pin="2"/>
 <wire x1="33.02" y1="27.94" x2="35.56" y2="27.94" width="0.1524" layer="91"/>
 <label x="33.02" y="27.94" size="1.778" layer="95"/>
@@
 <wire x1="256.54" y1="81.28" x2="256.54" y2="106.68" width="0.1524" layer="91"/>
 <wire x1="256.54" y1="106.68" x2="223.52" y2="106.68" width="0.1524" layer="91"/>
-<wire x1="223.52" y1="106.68" x2="218.44" y2="106.68" width="0.1524" layer="91"/>
+<wire x1="223.52" y1="106.68" x2="208.28" y2="106.68" width="0.1524" layer="91"/>
 <junction x="223.52" y="106.68"/>
-<label x="218.44" y="106.68" size="1.778" layer="95"/>
+<label x="200.66" y="106.68" size="1.778" layer="95"/>
+<pinref part="R5" gate="G$1" pin="1"/>
+<wire x1="208.28" y1="106.68" x2="200.66" y2="106.68" width="0.1524" layer="91"/>
+<junction x="208.28" y="106.68"/>
 </segment>
 </net>
@@
 <net name="D27" class="0">
 <segment>
-<pinref part="J5" gate="G$1" pin="2"/>
+<pinref part="J4" gate="G$1" pin="2"/>
 <wire x1="33.02" y1="15.24" x2="35.56" y2="15.24" width="0.1524" layer="91"/>
 <label x="33.02" y="15.24" size="1.778" layer="95"/>
@@
 <net name="D28" class="0">
 <segment>
-<pinref part="J6" gate="G$1" pin="1"/>
+<pinref part="J5" gate="G$1" pin="1"/>
 <wire x1="33.02" y1="25.4" x2="35.56" y2="25.4" width="0.1524" layer="91"/>
 <label x="33.02" y="25.4" size="1.778" layer="95"/>
@@
 </segment>
 <segment>
-<wire x1="200.66" y1="119.38" x2="271.78" y2="119.38" width="0.1524" layer="91" style="longdash"/>
-<wire x1="200.66" y1="119.38" x2="200.66" y2="22.86" width="0.1524" layer="91" style="longdash"/>
-<wire x1="200.66" y1="22.86" x2="271.78" y2="22.86" width="0.1524" layer="91" style="longdash"/>
+<wire x1="193.04" y1="119.38" x2="271.78" y2="119.38" width="0.1524" layer="91" style="longdash"/>
+<wire x1="193.04" y1="119.38" x2="193.04" y2="22.86" width="0.1524" layer="91" style="longdash"/>
+<wire x1="193.04" y1="22.86" x2="271.78" y2="22.86" width="0.1524" layer="91" style="longdash"/>
 <wire x1="271.78" y1="22.86" x2="271.78" y2="119.38" width="0.1524" layer="91" style="longdash"/>
 </segment>
@@
 </segment>
 </net>
+<net name="A5" class="0">
+<segment>
+<pinref part="MOTEINO_MEGA" gate="G$1" pin="A5"/>
+<wire x1="55.88" y1="124.46" x2="53.34" y2="124.46" width="0.1524" layer="91"/>
+<label x="53.34" y="124.46" size="1.778" layer="95"/>
+</segment>
+<segment>
+<pinref part="R5" gate="G$1" pin="2"/>
+<pinref part="R6" gate="G$1" pin="2"/>
+<wire x1="208.28" y1="96.52" x2="208.28" y2="91.44" width="0.1524" layer="91"/>
+<wire x1="208.28" y1="91.44" x2="208.28" y2="83.82" width="0.1524" layer="91"/>
+<wire x1="208.28" y1="91.44" x2="198.12" y2="91.44" width="0.1524" layer="91"/>
+<junction x="208.28" y="91.44"/>
+<label x="198.12" y="91.44" size="1.778" layer="95"/>
+</segment>
+</net>

Commit message: Added v0.61
Parts:
- added J6: 5V_GDN, SparkFun-Connectors:CONN_01
- added J9: 12-24V_VCC, SparkFun-Connectors:CONN_023.5MM-NO_SILK
- added R7: 50, SparkFun-Resistors:1MOHM-HORIZ_KIT-1/6W-5%
- J5: value DS18B20_12-24V_VCC -> DS18B20
Connections:
- new net N$7: J3.2, R7.1
- net 12-24V-VCC: now also J9.1; no longer J5.2
- net D26: now also R7.2; no longer J3.2
- net GND: now also J6.1, J9.2
Other:
- note added: "DS18B20"
- note removed: "DS18B20_VCC"
- moved on the sheet: J8, R5, R6
Changed lines of the file:
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@@
 <attributes>
 <attribute name="CNAME" value="MoteinoMega ABoatMon Sheild"/>
-<attribute name="CREVISION" value="0.6"/>
+<attribute name="CREVISION" value="0.61"/>
 <attribute name="DESIGNER" value="greg.cope@gmail.com"/>
 </attributes>
@@
 <part name="J3" library="SparkFun-Connectors" deviceset="CONN_02" device="3.5MM-NO_SILK" value="LED"/>
 <part name="J4" library="SparkFun-Connectors" deviceset="CONN_02" device="3.5MM-NO_SILK" value="DS18B20"/>
-<part name="J5" library="SparkFun-Connectors" deviceset="CONN_02" device="3.5MM-NO_SILK" value="DS18B20_12-24V_VCC"/>
+<part name="J5" library="SparkFun-Connectors" deviceset="CONN_02" device="3.5MM-NO_SILK" value="DS18B20"/>
 <part name="SUPPLY8" library="supply2" deviceset="GND" device=""/>
 <part name="Q2" library="transistor-power" deviceset="IRF9530" device="" value="IRF9Z14PBF"/>
@@
 <part name="R6" library="SparkFun-Resistors" deviceset="1MOHM" device="-HORIZ_KIT-1/6W-5%" value="3.3M"/>
 <part name="SUPPLY11" library="supply2" deviceset="GND" device=""/>
+<part name="J6" library="SparkFun-Connectors" deviceset="CONN_01" device="" value="5V_GDN"/>
+<part name="SUPPLY7" library="supply2" deviceset="GND" device=""/>
+<part name="J9" library="SparkFun-Connectors" deviceset="CONN_02" device="3.5MM-NO_SILK" value="12-24V_VCC"/>
+<part name="SUPPLY12" library="supply2" deviceset="GND" device=""/>
+<part name="R7" library="SparkFun-Resistors" deviceset="1MOHM" device="-HORIZ_KIT-1/6W-5%" value="50"/>
 </parts>
 <sheets>
 <sheet>
 <plain>
-<text x="23.622" y="34.036" size="1.778" layer="91">DS18B20_VCC</text>
+<text x="23.622" y="34.036" size="1.778" layer="91">DS18B20</text>
 <text x="218.44" y="114.3" size="1.778" layer="91">12V-24V to 5V Switched Regulator</text>
 <text x="15.24" y="170.18" size="1.778" layer="91">LED Button</text>
@@
 <instance part="J7" gate="J$1" x="238.76" y="43.18"/>
 <instance part="SUPPLY10" gate="GND" x="264.16" y="40.64"/>
-<instance part="J8" gate="G$1" x="205.74" y="27.94"/>
-<instance part="R5" gate="G$1" x="208.28" y="101.6" rot="R270"/>
-<instance part="R6" gate="G$1" x="208.28" y="78.74" rot="R90"/>
-<instance part="SUPPLY11" gate="GND" x="208.28" y="68.58"/>
+<instance part="J8" gate="G$1" x="203.2" y="27.94"/>
+<instance part="R5" gate="G$1" x="213.36" y="101.6" rot="R270"/>
+<instance part="R6" gate="G$1" x="213.36" y="78.74" rot="R90"/>
+<instance part="SUPPLY11" gate="GND" x="213.36" y="68.58"/>
+<instance part="J6" gate="G$1" x="203.2" y="40.64"/>
+<instance part="SUPPLY7" gate="GND" x="215.9" y="38.1"/>
+<instance part="J9" gate="G$1" x="195.58" y="106.68"/>
+<instance part="SUPPLY12" gate="GND" x="208.28" y="114.3" rot="R180"/>
+<instance part="R7" gate="G$1" x="30.48" y="142.24"/>
 </instances>
 <busses>
@@
 <segment>
 <pinref part="R6" gate="G$1" pin="1"/>
-<wire x1="208.28" y1="73.66" x2="208.28" y2="71.12" width="0.1524" layer="91"/>
+<wire x1="213.36" y1="73.66" x2="213.36" y2="71.12" width="0.1524" layer="91"/>
 <pinref part="SUPPLY11" gate="GND" pin="GND"/>
+</segment>
+<segment>
+<pinref part="J6" gate="G$1" pin="1"/>
+<wire x1="210.82" y1="40.64" x2="215.9" y2="40.64" width="0.1524" layer="91"/>
+<pinref part="SUPPLY7" gate="GND" pin="GND"/>
+</segment>
+<segment>
+<pinref part="J9" gate="G$1" pin="2"/>
+<wire x1="203.2" y1="109.22" x2="208.28" y2="109.22" width="0.1524" layer="91"/>
+<wire x1="208.28" y1="109.22" x2="208.28" y2="111.76" width="0.1524" layer="91"/>
+<pinref part="SUPPLY12" gate="GND" pin="GND"/>
 </segment>
 </net>
@@
 <net name="12-24V-VCC" class="0">
 <segment>
-<pinref part="J5" gate="G$1" pin="2"/>
-<wire x1="33.02" y1="27.94" x2="35.56" y2="27.94" width="0.1524" layer="91"/>
-<label x="33.02" y="27.94" size="1.778" layer="95"/>
-<label x="33.02" y="27.94" size="1.778" layer="95"/>
-<label x="33.02" y="27.94" size="1.778" layer="95"/>
-<label x="33.02" y="27.94" size="1.778" layer="95"/>
-<label x="33.02" y="27.94" size="1.778" layer="95"/>
-</segment>
-<segment>
 <pinref part="R4" gate="G$1" pin="2"/>
 <wire x1="223.52" y1="99.06" x2="223.52" y2="106.68" width="0.1524" layer="91"/>
@@
 <wire x1="256.54" y1="81.28" x2="256.54" y2="106.68" width="0.1524" layer="91"/>
 <wire x1="256.54" y1="106.68" x2="223.52" y2="106.68" width="0.1524" layer="91"/>
-<wire x1="223.52" y1="106.68" x2="208.28" y2="106.68" width="0.1524" layer="91"/>
+<wire x1="223.52" y1="106.68" x2="213.36" y2="106.68" width="0.1524" layer="91"/>
 <junction x="223.52" y="106.68"/>
-<label x="200.66" y="106.68" size="1.778" layer="95"/>
+<label x="218.44" y="106.68" size="1.778" layer="95"/>
 <pinref part="R5" gate="G$1" pin="1"/>
-<wire x1="208.28" y1="106.68" x2="200.66" y2="106.68" width="0.1524" layer="91"/>
-<junction x="208.28" y="106.68"/>
+<wire x1="213.36" y1="106.68" x2="203.2" y2="106.68" width="0.1524" layer="91"/>
+<junction x="213.36" y="106.68"/>
+<pinref part="J9" gate="G$1" pin="1"/>
+<junction x="203.2" y="106.68"/>
 </segment>
 </net>
@@
 </segment>
 <segment>
-<pinref part="J3" gate="G$1" pin="2"/>
-<wire x1="25.4" y1="142.24" x2="27.94" y2="142.24" width="0.1524" layer="91"/>
-<label x="25.4" y="142.24" size="1.778" layer="95"/>
+<pinref part="R7" gate="G$1" pin="2"/>
+<wire x1="35.56" y1="142.24" x2="40.64" y2="142.24" width="0.1524" layer="91"/>
+<label x="35.56" y="142.24" size="1.778" layer="95"/>
 </segment>
 </net>
@@
 </segment>
 <segment>
-<wire x1="193.04" y1="119.38" x2="271.78" y2="119.38" width="0.1524" layer="91" style="longdash"/>
-<wire x1="193.04" y1="119.38" x2="193.04" y2="22.86" width="0.1524" layer="91" style="longdash"/>
-<wire x1="193.04" y1="22.86" x2="271.78" y2="22.86" width="0.1524" layer="91" style="longdash"/>
+<wire x1="190.5" y1="119.38" x2="271.78" y2="119.38" width="0.1524" layer="91" style="longdash"/>
+<wire x1="190.5" y1="119.38" x2="190.5" y2="22.86" width="0.1524" layer="91" style="longdash"/>
+<wire x1="190.5" y1="22.86" x2="271.78" y2="22.86" width="0.1524" layer="91" style="longdash"/>
 <wire x1="271.78" y1="22.86" x2="271.78" y2="119.38" width="0.1524" layer="91" style="longdash"/>
 </segment>
@@
 <segment>
 <pinref part="J8" gate="G$1" pin="1"/>
-<wire x1="213.36" y1="27.94" x2="218.44" y2="27.94" width="0.1524" layer="91"/>
-<label x="213.36" y="27.94" size="1.778" layer="95"/>
+<wire x1="210.82" y1="27.94" x2="218.44" y2="27.94" width="0.1524" layer="91"/>
+<label x="210.82" y="27.94" size="1.778" layer="95"/>
 </segment>
 </net>
 <net name="N$3" class="0">
 <segment>
-<wire x1="10.16" y1="175.26" x2="38.1" y2="175.26" width="0.1524" layer="91" style="longdash"/>
-<wire x1="38.1" y1="175.26" x2="38.1" y2="124.46" width="0.1524" layer="91" style="longdash"/>
-<wire x1="38.1" y1="124.46" x2="10.16" y2="124.46" width="0.1524" layer="91" style="longdash"/>
+<wire x1="10.16" y1="175.26" x2="43.18" y2="175.26" width="0.1524" layer="91" style="longdash"/>
+<wire x1="43.18" y1="175.26" x2="43.18" y2="124.46" width="0.1524" layer="91" style="longdash"/>
+<wire x1="43.18" y1="124.46" x2="10.16" y2="124.46" width="0.1524" layer="91" style="longdash"/>
 <wire x1="10.16" y1="124.46" x2="10.16" y2="175.26" width="0.1524" layer="91" style="longdash"/>
 </segment>
@@
 <pinref part="R5" gate="G$1" pin="2"/>
 <pinref part="R6" gate="G$1" pin="2"/>
-<wire x1="208.28" y1="96.52" x2="208.28" y2="91.44" width="0.1524" layer="91"/>
-<wire x1="208.28" y1="91.44" x2="208.28" y2="83.82" width="0.1524" layer="91"/>
-<wire x1="208.28" y1="91.44" x2="198.12" y2="91.44" width="0.1524" layer="91"/>
-<junction x="208.28" y="91.44"/>
+<wire x1="213.36" y1="96.52" x2="213.36" y2="91.44" width="0.1524" layer="91"/>
+<wire x1="213.36" y1="91.44" x2="213.36" y2="83.82" width="0.1524" layer="91"/>
+<wire x1="213.36" y1="91.44" x2="198.12" y2="91.44" width="0.1524" layer="91"/>
+<junction x="213.36" y="91.44"/>
 <label x="198.12" y="91.44" size="1.778" layer="95"/>
 </segment>
 </net>
+<net name="N$7" class="0">
+<segment>
+<pinref part="J3" gate="G$1" pin="2"/>
+<pinref part="R7" gate="G$1" pin="1"/>
+</segment>
+</net>
