File: eagle/MoteinoMegaGPSSheild.brd (EAGLE design)
At the start: 58.1 x 33.6 mm, 32 parts, among them J1 BilgeSwitch, J2 Button, J3 LED, J4 DS18B20, J5 DS18B20, J6 GND, J7 OKI-78SR-5/1.5, J8 5V, J9 12-24V_VCC, Q1 NDP6020P, Q2 IRF9Z14PBF, Q3 2N7000, Q4 IRF9Z14PBF, Q5 2N7000

Commit message: eagle updates
Parts:
- removed D1: 1N5819-B, diode:DO41-7.6
- removed F1: 72V/0.25A, SparkFun-Fuses:PTH
- removed J1: BilgeSwitch, SparkFun-Connectors:SCREWTERMINAL-3.5MM-2-NS
- removed J2: Button, SparkFun-Connectors:SCREWTERMINAL-3.5MM-2-NS
- removed J3: LED, SparkFun-Connectors:SCREWTERMINAL-3.5MM-2-NS
- removed J4, J5: DS18B20, SparkFun-Connectors:SCREWTERMINAL-3.5MM-2-NS
- removed J6: GND, SparkFun-Connectors:1X01
- removed J7: OKI-78SR-5/1.5, SparkFun-Connectors:1X03
- removed J8: 5V, SparkFun-Connectors:1X01
- removed J9: 12-24V_VCC, SparkFun-Connectors:SCREWTERMINAL-3.5MM-2-NS
- removed JP2: FONA GSM, adafruit2:1X12-CB
- removed JP3: VCC_Bypass, jumper:JP1
- removed Q1: NDP6020P, transistor-power:TO220BV
- removed Q3, Q5: 2N7000, transistors:TO-92
- removed Q4: IRF9Z14PBF, transistor-power:TO220BV
- removed R1: 1k, SparkFun-Resistors:AXIAL-0.3
- removed R10, R8: 10k, SparkFun-Resistors:AXIAL-0.3
- removed R4, R9: 10K, SparkFun-Resistors:AXIAL-0.3
- added 5V: 5V, SparkFun-Connectors:1X02
- added C2: 0.1U, SparkFun-Capacitors:CAP-PTH-SMALL-KIT
- added FONA: (no value), SparkFun-Connectors:1X12
- added GND, GND_II: GND, SparkFun-Connectors:1X02
- added IO: (no value), SparkFun-Connectors:1X09
- added JST_PWR: VVC_5V, SparkFun-Connectors:JST-4-PTH
- added VCC: VCC, SparkFun-Connectors:1X02
- C1: value 0.1UF-KIT-EZ-50V-20% -> 0.1U
- Q2: value IRF9Z14PBF -> 60V/32A/35mΩ; device transistor-power:TO220BV -> SparkFun-DiscreteSemi:TO220V
- R5: value 27M -> 3.3M
- R6: value 3.3M -> 27M; device SparkFun-Resistors:AXIAL-0.3 -> adafruit:0309/12
- moved Q2 91.3 mm to (6.35, -43.2), turned to 0 degrees
- moved R5 88.3 mm to (5.08, -29.2), turned to 0 degrees
- moved R6 75.9 mm to (7.62, -14.0), turned to 0 degrees
- moved JP1 59.5 mm to (22.9, 2.54)
- moved R3 53.9 mm to (45.7, 8.89)
- moved R2 50.8 mm to (45.7, 11.4), turned to 0 degrees
- moved C1 43.6 mm to (39.4, 10.2), turned to 270 degrees
- moved R7 30.2 mm to (35.6, 12.7), turned to 270 degrees
- moved MOTEINO_MEGA 25.4 mm to (1.27, 30.5)
- moved JST1 17.1 mm to (2.54, 19.1), turned to 270 degrees
Connections:
- net D10_RX1 renamed D10_GPS_RX
- net D11_TX1 renamed D11_GPS_TX
- net D26 renamed D26_LED
- removed net 12-24V-SW: J7.3, Q2.D
- removed net 12-24V-VCC: F1.P$2, Q2.S, R4.P$2, R5.P$2
- removed net 5V_VCC: J7.1, J8.1
- removed net A5: MOTEINO_MEGA.A5, R5.P$1, R6.P$2
- removed net D12: MOTEINO_MEGA.D12, Q1.G, R1.P$1
- removed net D13_NETSTAT: JP2.2, MOTEINO_MEGA.D13
- removed net D14_KEY: JP2.6, MOTEINO_MEGA.D14
- removed net D18_PS: JP2.7, MOTEINO_MEGA.D18
- removed net D25: J2.2, MOTEINO_MEGA.A1
- removed net D27: J4.2, MOTEINO_MEGA.A3
- removed net D28: J5.1, MOTEINO_MEGA.A4
- removed net D3: J1.2, MOTEINO_MEGA.D3
- removed net D30: MOTEINO_MEGA.A6, R10.P$1
- removed net D8: JP2.4, MOTEINO_MEGA.D8
- removed net D9: JP2.3, MOTEINO_MEGA.D9
- removed net GPS_VCC: JP1.9, Q1.D
- removed net JUMPER: JP2.1, JP3.2, Q4.D
- removed net N$10: Q5.2, R10.P$2
- removed net N$5: Q4.G, Q5.3, R8.P$1
- removed net N$6: D1.A, J9.1
- removed net N$7: J3.2, R7.P$1
- removed net N$8: D1.C, F1.P$1
- removed net N$9: Q3.2, R9.P$2
- removed net SPEAKER2+: JP2.10
- new net 5V: 5V.1, 5V.2, JST_PWR.2
- new net A5_VCC_VD: C2.1, MOTEINO_MEGA.A5, R5.P$2, R6.1
- new net D12_GPS_MOS_N: MOTEINO_MEGA.D12, Q2.1
- new net D13_FONA_NETSTAT: FONA.2, MOTEINO_MEGA.D13
- new net D14_FONA_KEY: FONA.6, MOTEINO_MEGA.D14
- new net D18_FONA_PS: FONA.7, MOTEINO_MEGA.D18
- new net D25_LED_SWITCH: IO.9, MOTEINO_MEGA.A1
- new net D27_DS_PWR: IO.2, MOTEINO_MEGA.A3
- new net D28_DS_DATA: IO.3, MOTEINO_MEGA.A4
- new net D3_BILGESW: IO.5, MOTEINO_MEGA.D3
- new net D8_FONA_TX: FONA.3, MOTEINO_MEGA.D8
- new net D9_FONA_RX: FONA.4, MOTEINO_MEGA.D9
- new net N$1: JP1.3, Q2.2
- new net VCC: JST_PWR.4, R6.2, VCC.2
- net 3.3V: now also FONA.1, MOTEINO_MEGA.RST; no longer JP2.12, Q1.S, R1.P$2
- net D19_PWRON: now also VCC.1; no longer R9.P$1
- net GND: now also C2.2, FONA.11, GND.1, GND.2, GND_II.1, GND_II.2, IO.1, IO.4, IO.6, IO.8, JST_PWR.1, JST_PWR.3, Q2.3, R5.P$1; no longer J1.1, J2.1, J3.1, J4.1, J6.1, J7.2, J9.2, JP1.3, JP2.11, Q3.1, Q5.1, R6.P$1
- net N$2: now also IO.7, R7.P$1; no longer Q2.G, Q3.3, R4.P$1
- net VIN: now also FONA.12, MOTEINO_MEGA.VIN_2; no longer JP3.1, Q4.S, R8.P$2
Routing:
- net D9: track 107.9 -> 0.00 mm
- net 3.3V: track 81.7 -> 0.00 mm, vias 4 -> 0
- net VIN: track 78.8 -> 0.00 mm, vias 2 -> 0
- net N$2: track 62.1 -> 0.00 mm, vias 2 -> 0
- net D8: track 54.5 -> 0.00 mm, vias 1 -> 0
- net 12-24V-VCC: track 49.9 -> 0.00 mm, vias 1 -> 0
- net JUMPER: track 46.9 -> 0.00 mm, vias 4 -> 0
- net D19_PWRON: track 41.7 -> 0.00 mm
- net D13_NETSTAT: track 41.4 -> 0.00 mm
- net A0: track 40.5 -> 0.00 mm
- net D14_KEY: track 35.6 -> 0.00 mm, vias 1 -> 0
- net D10_GPS_RX: track 34.8 -> 0.00 mm
- net N$5: track 25.7 -> 0.00 mm, vias 1 -> 0
- net D12: track 25.0 -> 0.00 mm
- net D11_GPS_TX: track 25.0 -> 0.00 mm
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Other:
- board size 58.1 x 33.6 mm -> 57.5 x 31.1 mm
- board text added: "gregcope@gmail.com v1.99 MoteinoMega GPS Shield"
- board text removed: "+VE"
- board text removed: "0.1uF"
- board text removed: "12-24V"
- board text removed: "DQ"
- board text removed: "PIN"
- board text removed: "V0.999 MoteinoMega ABoatMon Shield gregcope@gmail.com"
- board text removed: "VDD"
