File: eagle/ABoatMon.brd (EAGLE design)
At the start: 78.7 x 61 mm, 29 parts, among them J1 5V, J2 GND, J3 GND, J4 5V, X1 MKDSN1,5/2-5,08

Commit message: DRC, ERC pass
Parts:
- renumbered J7 to JST
Other:
- board text added: "VIN LIPO"
Changed lines of the file:
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@@
 <text x="73.787" y="10.922" size="1.016" layer="25" font="vector" ratio="20">DS_PWR</text>
 <text x="73.787" y="16.129" size="1.016" layer="25" font="vector" ratio="20">DS_DA</text>
-<text x="62.484" y="58.674" size="1.016" layer="25" font="vector" ratio="20">VIN / LIPO</text>
+<text x="62.484" y="57.404" size="1.016" layer="25" font="vector" ratio="20">VIN
+LIPO</text>
 <text x="11.938" y="54.483" size="1.016" layer="25" font="vector" ratio="20" rot="R90">GND</text>
 <text x="13.462" y="57.15" size="1.016" layer="25" font="vector" ratio="20" rot="R270">VIN / LIPO</text>
@@
 <element name="U$7" library="microbuilder" package="MOUNTINGHOLE_2.5_PLATED" value="MOUNTINGHOLE2.5" x="65.024" y="49.53" smashed="yes"/>
 <element name="U$8" library="microbuilder" package="MOUNTINGHOLE_2.5_PLATED" value="MOUNTINGHOLE2.5" x="65.024" y="11.557" smashed="yes"/>
-<element name="J7" library="SparkFun-Connectors" library_urn="urn:adsk.eagle:library:513" package="1X09" package3d_urn="urn:adsk.eagle:package:38153/1" value="" x="72.39" y="6.35" smashed="yes" rot="R90">
+<element name="JST" library="SparkFun-Connectors" library_urn="urn:adsk.eagle:library:513" package="1X09" package3d_urn="urn:adsk.eagle:package:38153/1" value="" x="72.39" y="6.35" smashed="yes" rot="R90">
 <attribute name="NAME" x="70.993" y="5.08" size="0.6096" layer="25" font="vector" ratio="20" rot="R180"/>
 <attribute name="VALUE" x="74.422" y="5.08" size="0.6096" layer="27" font="vector" ratio="20" rot="R90"/>
@@
 <vertex x="8.89" y="48.26"/>
 </polygon>
-<contactref element="J7" pad="7"/>
-<contactref element="J7" pad="2"/>
-<contactref element="J7" pad="4"/>
-<contactref element="J7" pad="9"/>
+<contactref element="JST" pad="7"/>
+<contactref element="JST" pad="2"/>
+<contactref element="JST" pad="4"/>
+<contactref element="JST" pad="9"/>
 <contactref element="X1" pad="2"/>
 <via x="21.59" y="45.72" extent="1-16" drill="0.508"/>
@@
 <wire x1="2.286" y1="27.686" x2="3.81" y2="29.21" width="0.6096" layer="1"/>
 <wire x1="2.794" y1="27.178" x2="2.286" y2="27.686" width="0.6096" layer="1"/>
-<wire x1="2.794" y1="21.336" x2="2.794" y2="27.178" width="0.6096" layer="1"/>
-<wire x1="5.08" y1="19.05" x2="2.794" y2="21.336" width="0.6096" layer="1"/>
-<wire x1="5.08" y1="19.05" x2="5.055" y2="19.0289" width="0.6096" layer="1"/>
+<wire x1="2.794" y1="20.701" x2="2.794" y2="27.178" width="0.6096" layer="1"/>
+<wire x1="5.055" y1="19.0289" x2="4.4661" y2="19.0289" width="0.6096" layer="1"/>
+<wire x1="4.4661" y1="19.0289" x2="2.794" y2="20.701" width="0.6096" layer="1"/>
 </signal>
 <signal name="5V" class="1">
@@
 <signal name="D25_LED_SWITCH">
 <contactref element="MOTEINO_MEGA" pad="A1"/>
-<contactref element="J7" pad="6"/>
+<contactref element="JST" pad="6"/>
 <wire x1="41.91" y1="57.912" x2="41.91" y2="58.547" width="0.6096" layer="16"/>
 <wire x1="48.514" y1="51.308" x2="41.91" y2="57.912" width="0.6096" layer="16"/>
@@
 <signal name="D3_BILGESW">
 <contactref element="MOTEINO_MEGA" pad="D3"/>
-<contactref element="J7" pad="1"/>
+<contactref element="JST" pad="1"/>
 <wire x1="29.21" y1="57.912" x2="29.21" y2="58.547" width="0.6096" layer="16"/>
 <wire x1="32.766" y1="54.356" x2="29.21" y2="57.912" width="0.6096" layer="16"/>
@@
 <signal name="D28_DS_DATA">
 <contactref element="MOTEINO_MEGA" pad="A4"/>
-<contactref element="J7" pad="5"/>
+<contactref element="JST" pad="5"/>
 <wire x1="49.53" y1="57.912" x2="49.53" y2="58.547" width="0.6096" layer="16"/>
 <wire x1="59.436" y1="48.006" x2="49.53" y2="57.912" width="0.6096" layer="16"/>
@@
 <signal name="D27_DS_PWR">
 <contactref element="MOTEINO_MEGA" pad="A3"/>
-<contactref element="J7" pad="3"/>
+<contactref element="JST" pad="3"/>
 <wire x1="46.99" y1="57.912" x2="46.99" y2="58.547" width="0.6096" layer="16"/>
 <wire x1="57.404" y1="47.498" x2="46.99" y2="57.912" width="0.6096" layer="16"/>
@@
 </signal>
 <signal name="LED">
-<contactref element="J7" pad="8"/>
+<contactref element="JST" pad="8"/>
 <contactref element="R7" pad="P$1"/>
 <wire x1="71.628" y1="24.13" x2="72.39" y2="24.13" width="0.6096" layer="1"/>
@@
 <mfgpreviewcolor name="substratecolor" color="0xFF786E46"/>
 </mfgpreviewcolors>
-<errors>
-</errors>
 </board>
 </drawing>
