File: eagle/ABoatMon.sch (EAGLE design)
At the start: 29 parts, among them J1 5V, J2 GND, J3 GND, J4 5V, X1 MKDSN1,5/2-5,08

Commit message: removed extra 3.3v labels
Changed lines of the file:
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@@
 <segment>
 <label x="180.34" y="63.5" size="1.778" layer="95" rot="R90"/>
-<wire x1="180.34" y1="78.74" x2="180.34" y2="50.8" width="0.1524" layer="91"/>
+<wire x1="180.34" y1="78.74" x2="180.34" y2="63.5" width="0.1524" layer="91"/>
 <pinref part="VCC" gate="G$1" pin="2"/>
 <wire x1="170.18" y1="78.74" x2="180.34" y2="78.74" width="0.1524" layer="91"/>

Commit message: message logic
Parts:
- added J5: (no value), SparkFun-Connectors:CONN_04JST-PTH
Connections:
- new net D16_SCL: J5.3, MOTEINO_MEGA.D16_SCL
- new net D17_SDA: J5.4, MOTEINO_MEGA.D17_SDA
- new net D20_OLED_VCC: J5.2, MOTEINO_MEGA.D20
- net GND: now also J5.1
Changed lines of the file:
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@@
 <part name="X1" library="con-phoenix-508" library_urn="urn:adsk.eagle:library:176" deviceset="MKDSN1,5/2-5,08" device="" package3d_urn="urn:adsk.eagle:package:9630/1"/>
 <part name="R1" library="SparkFun-Resistors" deviceset="1KOHM" device="-HORIZ-1/4W-1%" value="4.7K"/>
+<part name="J5" library="SparkFun-Connectors" library_urn="urn:adsk.eagle:library:513" deviceset="CONN_04" device="JST-PTH" package3d_urn="urn:adsk.eagle:package:38101/1"/>
 </parts>
 <sheets>
@@
 <attribute name="VALUE" x="255.524" y="129.54" size="1.778" layer="96" font="vector" rot="R90" align="top-center"/>
 </instance>
+<instance part="J5" gate="G$1" x="210.82" y="104.14" smashed="yes">
+<attribute name="VALUE" x="205.74" y="96.774" size="1.778" layer="96" font="vector"/>
+<attribute name="NAME" x="205.74" y="112.268" size="1.778" layer="95" font="vector"/>
+</instance>
 </instances>
 <busses>
@@
 <label x="215.9" y="144.78" size="1.778" layer="95"/>
 </segment>
+<segment>
+<pinref part="J5" gate="G$1" pin="1"/>
+<wire x1="215.9" y1="101.6" x2="236.22" y2="101.6" width="0.1524" layer="91"/>
+<label x="215.9" y="101.6" size="1.778" layer="95"/>
+</segment>
 </net>
 <net name="VIN" class="1">
@@
 </segment>
 </net>
+<net name="D17_SDA" class="0">
+<segment>
+<pinref part="MOTEINO_MEGA" gate="G$1" pin="D17_SDA"/>
+<wire x1="106.68" y1="147.32" x2="111.76" y2="147.32" width="0.1524" layer="91"/>
+<label x="106.68" y="147.32" size="1.778" layer="95"/>
+</segment>
+<segment>
+<pinref part="J5" gate="G$1" pin="4"/>
+<wire x1="215.9" y1="109.22" x2="236.22" y2="109.22" width="0.1524" layer="91"/>
+<label x="215.9" y="109.22" size="1.778" layer="95"/>
+</segment>
+</net>
+<net name="D16_SCL" class="0">
+<segment>
+<pinref part="MOTEINO_MEGA" gate="G$1" pin="D16_SCL"/>
+<wire x1="106.68" y1="144.78" x2="111.76" y2="144.78" width="0.1524" layer="91"/>
+<label x="106.68" y="144.78" size="1.778" layer="95"/>
+</segment>
+<segment>
+<pinref part="J5" gate="G$1" pin="3"/>
+<wire x1="215.9" y1="106.68" x2="236.22" y2="106.68" width="0.1524" layer="91"/>
+<label x="215.9" y="106.68" size="1.778" layer="95"/>
+</segment>
+</net>
+<net name="D20_OLED_VCC" class="0">
+<segment>
+<pinref part="MOTEINO_MEGA" gate="G$1" pin="D20"/>
+<wire x1="106.68" y1="154.94" x2="111.76" y2="154.94" width="0.1524" layer="91"/>
+<label x="106.68" y="154.94" size="1.778" layer="95"/>
+</segment>
+<segment>
+<pinref part="J5" gate="G$1" pin="2"/>
+<wire x1="215.9" y1="104.14" x2="236.22" y2="104.14" width="0.1524" layer="91"/>
+<label x="215.9" y="104.14" size="1.778" layer="95"/>
+</segment>
+</net>

Commit message: v0.959 board layout, moved to 0.1 not jst
Parts:
- removed J5: (no value), SparkFun-Connectors:CONN_04JST-PTH
- added J7: (no value), SparkFun-Connectors:CONN_05NO_SILK
Connections:
- new net D21_SPARE: J7.1, MOTEINO_MEGA.D21
- net D16_SCL: now also J7.4; no longer J5.3
- net D17_SDA: now also J7.5; no longer J5.4
- net D20_OLED_VCC: now also J7.3; no longer J5.2
- net GND: now also J7.2; no longer J5.1
Changed lines of the file:
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@@
 <attributes>
 <attribute name="CNAME" value="MoteinoMega ABoatMon Shield"/>
-<attribute name="CREVISION" value="0.949"/>
+<attribute name="CREVISION" value="0.959"/>
 <attribute name="DESIGNER" value="gregcope@gmail.com"/>
 </attributes>
@@
 <part name="X1" library="con-phoenix-508" library_urn="urn:adsk.eagle:library:176" deviceset="MKDSN1,5/2-5,08" device="" package3d_urn="urn:adsk.eagle:package:9630/1"/>
 <part name="R1" library="SparkFun-Resistors" deviceset="1KOHM" device="-HORIZ-1/4W-1%" value="4.7K"/>
-<part name="J5" library="SparkFun-Connectors" library_urn="urn:adsk.eagle:library:513" deviceset="CONN_04" device="JST-PTH" package3d_urn="urn:adsk.eagle:package:38101/1"/>
+<part name="J7" library="SparkFun-Connectors" library_urn="urn:adsk.eagle:library:513" deviceset="CONN_05" device="NO_SILK" package3d_urn="urn:adsk.eagle:package:38108/1"/>
 </parts>
 <sheets>
@@
 <attribute name="VALUE" x="255.524" y="129.54" size="1.778" layer="96" font="vector" rot="R90" align="top-center"/>
 </instance>
-<instance part="J5" gate="G$1" x="210.82" y="104.14" smashed="yes">
-<attribute name="VALUE" x="205.74" y="96.774" size="1.778" layer="96" font="vector"/>
+<instance part="J7" gate="G$1" x="208.28" y="104.14" smashed="yes">
+<attribute name="VALUE" x="205.74" y="94.234" size="1.778" layer="96" font="vector"/>
 <attribute name="NAME" x="205.74" y="112.268" size="1.778" layer="95" font="vector"/>
 </instance>
@@
 </segment>
 <segment>
-<pinref part="J5" gate="G$1" pin="1"/>
 <wire x1="215.9" y1="101.6" x2="236.22" y2="101.6" width="0.1524" layer="91"/>
 <label x="215.9" y="101.6" size="1.778" layer="95"/>
+<pinref part="J7" gate="G$1" pin="2"/>
 </segment>
 </net>
@@
 </segment>
 <segment>
-<pinref part="J5" gate="G$1" pin="4"/>
 <wire x1="215.9" y1="109.22" x2="236.22" y2="109.22" width="0.1524" layer="91"/>
 <label x="215.9" y="109.22" size="1.778" layer="95"/>
+<pinref part="J7" gate="G$1" pin="5"/>
 </segment>
 </net>
@@
 </segment>
 <segment>
-<pinref part="J5" gate="G$1" pin="3"/>
 <wire x1="215.9" y1="106.68" x2="236.22" y2="106.68" width="0.1524" layer="91"/>
 <label x="215.9" y="106.68" size="1.778" layer="95"/>
+<pinref part="J7" gate="G$1" pin="4"/>
 </segment>
 </net>
@@
 </segment>
 <segment>
-<pinref part="J5" gate="G$1" pin="2"/>
 <wire x1="215.9" y1="104.14" x2="236.22" y2="104.14" width="0.1524" layer="91"/>
 <label x="215.9" y="104.14" size="1.778" layer="95"/>
-</segment>
-</net>
+<pinref part="J7" gate="G$1" pin="3"/>
+</segment>
+</net>
+<net name="D21_SPARE" class="0">
+<segment>
+<pinref part="MOTEINO_MEGA" gate="G$1" pin="D21"/>
+<wire x1="106.68" y1="157.48" x2="111.76" y2="157.48" width="0.1524" layer="91"/>
+<label x="106.68" y="157.48" size="1.778" layer="95"/>
+</segment>
+<segment>
+<pinref part="J7" gate="G$1" pin="1"/>
+<wire x1="215.9" y1="99.06" x2="236.22" y2="99.06" width="0.1524" layer="91"/>
+<label x="215.9" y="99.06" size="1.778" layer="95"/>
+</segment>
+</net>
